File: PCB/Capstone/Capstone.kicad_sch (KiCad schematic)
At the start: 3 parts, among them J1 ESP_Left, J2 ESP_Right, J3 TFT

Commit message: Added PCB components
Connections:
- net CTP_INT: now also J2.6 (Pin_6); no longer J2.8 (Pin_8)
Changed lines of the file:
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@@
+	(wire
+		(pts
+			(xy 119.38 74.93) (xy 120.65 74.93)
+		)
+		(stroke
+			(width 0)
+			(type default)
+		)
+	)
 	(wire
 		(pts
@@
 		(pts
 			(xy 146.05 71.12) (xy 153.67 71.12)
+		)
+		(stroke
+			(width 0)
+			(type default)
+		)
+	)
+	(wire
+		(pts
+			(xy 119.38 77.47) (xy 120.65 77.47)
 		)
 		(stroke
@@
 	)
 	(label "CTP_RST"
-		(at 119.38 74.93 0)
+		(at 120.65 74.93 0)
 		(effects
 			(font
@@
 	)
 	(label "CTP_INT"
-		(at 119.38 72.39 0)
-		(effects
-			(font
+		(at 120.65 77.47 0)
+		(effects
+			(font
